Commit message: add collision mesh and delete mimic joint

File: inmoov_description/urdf/asmHand.urdf.xacro (robot description, xacro)
@@ -11,4 +11,10 @@
         <xacro:frame_color/>
       </visual>
+      <collision>
+        <geometry>
+          <mesh filename="package://inmoov_meshes/meshes/${side}_hand.stl" scale="0.001 0.001 0.001"/>
+        </geometry>
+        <origin rpy="0 0 0" xyz="0 0 0"/>
+      </collision>
       <xacro:if value="${side == 'l'}">
         <xacro:l_hand_inertial/>
@@ -26,4 +32,10 @@
         <xacro:frame_color/>
       </visual>
+      <collision>
+        <geometry>
+          <mesh filename="package://inmoov_meshes/meshes/${side}_thumb5_1.stl" scale="0.001 0.001 0.001"/>
+        </geometry>
+        <origin rpy="0 0 0" xyz="0 0 0"/>
+      </collision>
       <xacro:if value="${side == 'l'}">
         <xacro:l_thumb5_1_inertial/>
@@ -41,4 +53,10 @@
         <xacro:frame_color/>
       </visual>
+      <collision>
+        <geometry>
+          <mesh filename="package://inmoov_meshes/meshes/thumb5_2.stl" scale="0.001 0.001 0.001"/>
+        </geometry>
+        <origin rpy="0 0 0" xyz="0 0 0"/>
+      </collision>
       <xacro:thumb5_2_inertial/>
     </link>
@@ -51,4 +69,10 @@
         <xacro:frame_color/>
       </visual>
+      <collision>
+        <geometry>
+          <mesh filename="package://inmoov_meshes/meshes/thumb5_3.stl" scale="0.001 0.001 0.001"/>
+        </geometry>
+        <origin rpy="0 0 0" xyz="0 0 0"/>
+      </collision>
       <xacro:thumb5_3_inertial/>
     </link>
@@ -61,4 +85,9 @@
         <xacro:frame_color/>
       </visual>
+      <collision>
+        <mesh filename="package://inmoov_meshes/meshes/index3_1.stl" scale="0.001 0.001 0.001"/>
+        </geometry>
+        <origin rpy="0 0 0" xyz="0 0 0"/>
+      </collision>
       <xacro:index3_1_inertial/>
     </link>
@@ -71,4 +100,10 @@
         <xacro:frame_color/>
       </visual>
+      <collision>
+        <geometry>
+          <mesh filename="package://inmoov_meshes/meshes/index3_2.stl" scale="0.001 0.001 0.001"/>
+        </geometry>
+        <origin rpy="0 0 0" xyz="0 0 0"/>
+      </collision>
       <xacro:index3_2_inertial/>
     </link>
@@ -81,4 +116,10 @@
         <xacro:frame_color/>
       </visual>
+      <collision>
+        <geometry>
+          <mesh filename="package://inmoov_meshes/meshes/index3_3.stl" scale="0.001 0.001 0.001"/>
+        </geometry>
+        <origin rpy="0 0 0" xyz="0 0 0"/>
+      </collision>
       <xacro:index3_3_inertial/>
     </link>
@@ -91,4 +132,10 @@
         <xacro:frame_color/>
       </visual>
+      <collision>
+        <geometry>
+          <mesh filename="package://inmoov_meshes/meshes/middle3_1.stl" scale="0.001 0.001 0.001"/>
+        </geometry>
+        <origin rpy="0 0 0" xyz="0 0 0"/>
+      </collision>
       <xacro:middle3_1_inertial/>
     </link>
@@ -101,4 +148,10 @@
         <xacro:frame_color/>
       </visual>
+      <collision>
+        <geometry>
+          <mesh filename="package://inmoov_meshes/meshes/middle3_2.stl" scale="0.001 0.001 0.001"/>
+        </geometry>
+        <origin rpy="0 0 0" xyz="0 0 0"/>
+      </collision>
       <xacro:middle3_2_inertial/>
     </link>
@@ -111,4 +164,10 @@
         <xacro:frame_color/>
       </visual>
+      <collision>
+        <geometry>
+          <mesh filename="package://inmoov_meshes/meshes/middle3_3.stl" scale="0.001 0.001 0.001"/>
+        </geometry>
+        <origin rpy="0 0 0" xyz="0 0 0"/>
+      </collision>
       <xacro:middle3_3_inertial/>
     </link>
@@ -121,4 +180,10 @@
         <xacro:frame_color/>
       </visual>
+      <collision>
+        <geometry>
+          <mesh filename="package://inmoov_meshes/meshes/${side}_ring3_1.stl" scale="0.001 0.001 0.001"/>
+        </geometry>
+        <origin rpy="0 0 0" xyz="0 0 0"/>
+      </collision>
       <xacro:if value="${side == 'l'}">
         <xacro:l_ring3_1_inertial/>
@@ -136,4 +201,10 @@
         <xacro:frame_color/>
       </visual>
+      <collision>
+        <geometry>
+          <mesh filename="package://inmoov_meshes/meshes/ring3_2.stl" scale="0.001 0.001 0.001"/>
+        </geometry>
+        <origin rpy="0 0 0" xyz="0 0 0"/>
+      </collision>
       <xacro:ring3_2_inertial/>
     </link>
@@ -146,4 +217,10 @@
         <xacro:frame_color/>
       </visual>
+      <collision>
+        <geometry>
+          <mesh filename="package://inmoov_meshes/meshes/ring3_3.stl" scale="0.001 0.001 0.001"/>
+        </geometry>
+        <origin rpy="0 0 0" xyz="0 0 0"/>
+      </collision>
       <xacro:ring3_3_inertial/>
     </link>
@@ -156,4 +233,10 @@
         <xacro:frame_color/>
       </visual>
+      <collision>
+        <geometry>
+          <mesh filename="package://inmoov_meshes/meshes/ring3_4.stl" scale="0.001 0.001 0.001"/>
+        </geometry>
+        <origin rpy="0 0 0" xyz="0 0 0"/>
+      </collision>
       <xacro:ring3_4_inertial/>
     </link>
@@ -166,4 +249,10 @@
         <xacro:frame_color/>
       </visual>
+      <collision>
+        <geometry>
+          <mesh filename="package://inmoov_meshes/meshes/${side}_pinky3_1.stl" scale="0.001 0.001 0.001"/>
+        </geometry>
+        <origin rpy="0 0 0" xyz="0 0 0"/>
+      </collision>
       <xacro:if value="${side == 'l'}">
         <xacro:l_pinky3_1_inertial/>
@@ -181,4 +270,10 @@
         <xacro:frame_color/>
       </visual>
+      <collision>
+        <geometry>
+          <mesh filename="package://inmoov_meshes/meshes/pinky3_2.stl" scale="0.001 0.001 0.001"/>
+        </geometry>
+        <origin rpy="0 0 0" xyz="0 0 0"/>
+      </collision>
       <xacro:pinky3_2_inertial/>
     </link>
@@ -191,4 +286,10 @@
         <xacro:frame_color/>
       </visual>
+      <collision>
+        <geometry>
+          <mesh filename="package://inmoov_meshes/meshes/pinky3_3.stl" scale="0.001 0.001 0.001"/>
+        </geometry>
+        <origin rpy="0 0 0" xyz="0 0 0"/>
+      </collision>
       <xacro:pinky3_3_inertial/>
     </link>
@@ -201,4 +302,10 @@
         <xacro:frame_color/>
       </visual>
+      <collision>
+        <geometry>
+          <mesh filename="package://inmoov_meshes/meshes/pinky3_4.stl" scale="0.001 0.001 0.001"/>
+        </geometry>
+        <origin rpy="0 0 0" xyz="0 0 0"/>
+      </collision>
       <xacro:pinky3_4_inertial/>
     </link>
@@ -212,5 +319,4 @@
         </xacro:if>
       <origin rpy="${flip * 0.1} 0 0" xyz="0 ${flip * 0.029} -0.0577"/>
-      <mimic joint="${side}_thumb_joint" multiplier="${flip *0.75}" offset="0"/>
       <parent link="${side}_hand_link"/>
       <child link="${side}_thumb1_link"/>
@@ -237,5 +343,4 @@
         </xacro:if>
       <origin rpy="0 0 0" xyz="0 0 -0.035"/>
-      <mimic joint="${side}_thumb_joint" multiplier="1" offset="0"/>
       <parent link="${side}_thumb2_link"/>
       <child link="${side}_thumb3_link"/>
@@ -250,5 +355,4 @@
         </xacro:if>
       <origin rpy="${flip * 0.1} 0 0" xyz="-0.0015 ${flip * 0.0342}  -0.119"/>
-      <mimic joint="${side}_index_joint" multiplier="1" offset="0"/>
       <parent link="${side}_hand_link"/>
       <child link="${side}_index1_link"/>
@@ -275,5 +379,4 @@
         </xacro:if>
       <origin rpy="0 0 0" xyz="0 0 -0.024"/>
-      <mimic joint="${side}_index_joint" multiplier="1" offset="0"/>
       <parent link="${side}_index2_link"/>
       <child link="${side}_index3_link"/>
@@ -288,5 +391,4 @@
         </xacro:if>
       <origin rpy="0 0 0" xyz="-0.00175 ${flip * 0.007}  -0.12325"/>
-      <mimic joint="${side}_middle_joint" multiplier="1" offset="0"/>
       <parent link="${side}_hand_link"/>
       <child link="${side}_middle1_link"/>
@@ -313,5 +415,4 @@
         </xacro:if>
       <origin rpy="0 0 0" xyz="0 0.0005 -0.0259"/>
-      <mimic joint="${side}_middle_joint" multiplier="1" offset="0"/>
       <parent link="${side}_middle2_link"/>
       <child link="${side}_middle3_link"/>
@@ -326,5 +427,4 @@
         </xacro:if>
       <origin rpy="${flip * 0.7} 0 0" xyz="0 ${flip * -0.00705} -0.0794"/>
-      <mimic joint="${side}_ring_joint" multiplier="${flip * -0.1}" offset="0"/>
       <parent link="${side}_hand_link"/>
       <child link="${side}_ring1_link"/>
@@ -351,5 +451,4 @@
         </xacro:if>
       <origin rpy="0 0 0" xyz="0 0.0005 -0.0345"/>
-      <mimic joint="${side}_ring_joint" multiplier="1" offset="0"/>
       <parent link="${side}_ring2_link"/>
       <child link="${side}_ring3_link"/>
@@ -364,5 +463,4 @@
         </xacro:if>
       <origin rpy="0 0 0" xyz="0 0.0004 -0.0229"/>
-      <mimic joint="${side}_ring_joint" multiplier="1" offset="0"/>
       <parent link="${side}_ring3_link"/>
       <child link="${side}_ring4_link"/>
@@ -377,5 +475,4 @@
         </xacro:if>
       <origin rpy="${flip * 0.7} 0 0" xyz="0 ${flip * -0.0270} -0.0555"/>
-      <mimic joint="${side}_pinky_joint" multiplier="${flip * -0.1}" offset="0"/>
       <parent link="${side}_hand_link"/>
       <child link="${side}_pinky1_link"/>
@@ -402,5 +499,4 @@
         </xacro:if>
       <origin rpy="0 0 0" xyz="0 0.0005 -0.031"/>
-      <mimic joint="${side}_pinky_joint" multiplier="1" offset="0"/>
       <parent link="${side}_pinky2_link"/>
       <child link="${side}_pinky3_link"/>
@@ -415,5 +511,4 @@
         </xacro:if>
       <origin rpy="0 0 0" xyz="0 0.0004 -0.0208"/>
-      <mimic joint="${side}_pinky_joint" multiplier="1" offset="0"/>
       <parent link="${side}_pinky3_link"/>
       <child link="${side}_pinky4_link"/>
@@ -427,4 +522,10 @@
         <xacro:cover_color/>
       </visual>
+      <collision>
+        <geometry>
+          <mesh filename="package://inmoov_meshes/meshes/${side}_cover_hand.stl" scale="0.001 0.001 0.001"/>
+        </geometry>
+        <origin rpy="0 0 0" xyz="0 0 0"/>
+      </collision>
       <xacro:if value="${side == 'l'}">
         <xacro:l_cover_hand_inertial/>
@@ -442,4 +543,10 @@
         <xacro:cover_color/>
       </visual>
+      <collision>
+        <geometry>
+          <mesh filename="package://inmoov_meshes/meshes/${side}_cover_handring.stl" scale="0.001 0.001 0.001"/>
+        </geometry>
+        <origin rpy="0 0 0" xyz="0 0 0"/>
+      </collision>
       <xacro:if value="${side == 'l'}">
         <xacro:l_cover_handring_inertial/>
@@ -457,4 +564,10 @@
         <xacro:cover_color/>
       </visual>
+      <collision>
+        <geometry>
+          <mesh filename="package://inmoov_meshes/meshes/${side}_cover_handpinky.stl" scale="0.001 0.001 0.001"/>
+        </geometry>
+        <origin rpy="0 0 0" xyz="0 0 0"/>
+      </collision>
       <xacro:if value="${side == 'l'}">
         <xacro:l_cover_handpinky_inertial/>
@@ -472,4 +585,10 @@
         <xacro:cover_color/>
       </visual>
+      <collision>
+        <geometry>
+          <mesh filename="package://inmoov_meshes/meshes/${side}_cover_thumb.stl" scale="0.001 0.001 0.001"/>
+        </geometry>
+        <origin rpy="0 0 0" xyz="0 0 0"/>
+      </collision>
       <xacro:if value="${side == 'l'}">
         <xacro:l_cover_thumb_inertial/>
@@ -487,4 +606,10 @@
         <xacro:cover_color/>
       </visual>
+      <collision>
+        <geometry>
+          <mesh filename="package://inmoov_meshes/meshes/${side}_cover_index.stl" scale="0.001 0.001 0.001"/>
+        </geometry>
+        <origin rpy="0 0 0" xyz="0 0 0"/>
+      </collision>
       <xacro:if value="${side == 'l'}">
         <xacro:l_cover_index_inertial/>
@@ -502,4 +627,10 @@
         <xacro:cover_color/>
       </visual>
+      <collision>
+        <geometry>
+          <mesh filename="package://inmoov_meshes/meshes/${side}_cover_middle.stl" scale="0.001 0.001 0.001"/>
+        </geometry>
+        <origin rpy="0 0 0" xyz="0 0 0"/>
+      </collision>
       <xacro:if value="${side == 'l'}">
         <xacro:l_cover_middle_inertial/>
@@ -517,4 +648,10 @@
         <xacro:cover_color/>
       </visual>
+      <collision>
+        <geometry>
+          <mesh filename="package://inmoov_meshes/meshes/${side}_cover_ring.stl" scale="0.001 0.001 0.001"/>
+        </geometry>
+        <origin rpy="0 0 0" xyz="0 0 0"/>
+      </collision>
       <xacro:if value="${side == 'l'}">
         <xacro:l_cover_ring_inertial/>
@@ -532,4 +669,10 @@
         <xacro:cover_color/>
       </visual>
+      <collision>
+        <geometry>
+          <mesh filename="package://inmoov_meshes/meshes/${side}_cover_pinky.stl" scale="0.001 0.001 0.001"/>
+        </geometry>
+        <origin rpy="0 0 0" xyz="0 0 0"/>
+      </collision>
       <xacro:if value="${side == 'l'}">
         <xacro:l_cover_pinky_inertial/>

Commit message: bug fix

File: inmoov_description/urdf/asmHand.urdf.xacro (robot description, xacro)
@@ -86,5 +86,6 @@
       </visual>
       <collision>
-        <mesh filename="package://inmoov_meshes/meshes/index3_1.stl" scale="0.001 0.001 0.001"/>
+        <geometry>
+          <mesh filename="package://inmoov_meshes/meshes/index3_1.stl" scale="0.001 0.001 0.001"/>
         </geometry>
         <origin rpy="0 0 0" xyz="0 0 0"/>
