Commit message: new inmoov shadow hand with ball joint

File: inmoov_description/urdf/asmArm.urdf.xacro (robot description, xacro)
@@ -34,4 +34,6 @@
     </xacro:if>
   </link>
+  <link name="${side}_bicep_link_aux_0"/>
+  <link name="${side}_bicep_link_aux_1"/>
   <link name="${side}_bicep_link">
     <visual>
@@ -63,10 +65,10 @@
       <xacro:cover_color/>
     </visual>
-    <collision>
+    <!-- <collision>
       <geometry>
         <cylinder length="0.28" radius="0.045"/>
       </geometry>
       <origin rpy="0 0 0" xyz="-0.00 0 -0.14"/>
-    </collision>
+    </collision> -->
     <xacro:if value="${side == 'l'}">
       <xacro:l_forearm_inertial/>
@@ -76,4 +78,17 @@
     </xacro:if>
   </link>
+  <joint name="${side}_shoulder_lift_joint_old" type="fixed">
+    <origin rpy="0 0 0" xyz="0 ${flip * -0.012} -0.04"/>
+    <parent link="${side}_shoulder_base_link"/>
+    <child link="${side}_shoulder_link"/>
+  </joint>
+  <joint name="${side}_shoulder_out_joint" type="revolute">
+    <axis xyz="1 0 0"/>
+    <limit effort="1000.0" lower="-1.57079632679" upper="1.57079632679" velocity="1745.32925199"/>
+    <!-- <origin rpy="0 0 0" xyz="0 0 0"/> -->
+    <origin rpy="0 0 0" xyz="0 ${flip * -0.066} -0.06"/>
+    <parent link="${side}_shoulder_link"/>
+    <child link="${side}_bicep_link_aux_0"/>
+  </joint>
   <joint name="${side}_shoulder_lift_joint" type="revolute">
     <axis xyz="0 1 0"/>
@@ -84,7 +99,7 @@
       <limit effort="1000.0" lower="${r_shoulder_lift_joint_lower}" upper="${r_shoulder_lift_joint_upper}" velocity="${r_shoulder_lift_joint_velocity}" />
     </xacro:if>
-    <origin rpy="0 0 0" xyz="0 ${flip * -0.012} -0.04"/>
-    <parent link="${side}_shoulder_base_link"/>
-    <child link="${side}_shoulder_link"/>
+    <origin rpy="0 0 0" xyz="0 0 0"/>
+    <parent link="${side}_bicep_link_aux_0"/>
+    <child link="${side}_bicep_link_aux_1"/>
   </joint>
   <joint name="${side}_upper_arm_roll_joint" type="revolute">
@@ -96,6 +111,6 @@
       <limit effort="1000.0" lower="${r_upper_arm_roll_joint_lower}" upper="${r_upper_arm_roll_joint_upper}" velocity="${r_upper_arm_roll_joint_velocity}" />
     </xacro:if>
-    <origin rpy="0 0 0" xyz="0 ${flip * -0.066} -0.06"/>
-    <parent link="${side}_shoulder_link"/>
+    <origin rpy="0 0 0" xyz="0 0 0"/>
+    <parent link="${side}_bicep_link_aux_1"/>
     <child link="${side}_bicep_link"/>
   </joint>

File: inmoov_description/urdf/asmEye.urdf.xacro (robot description, xacro)
@@ -17,5 +17,5 @@
     </xacro:if>
   </link>
-  <link name="${side}_camera_link">
+  <!-- <link name="${side}_camera_link">
     <visual>
       <geometry>
@@ -26,5 +26,5 @@
     </visual>
     <xacro:camera_inertial/>
-  </link>
+  </link> -->
   <link name="${side}_eye_link">
     <visual>
@@ -47,9 +47,9 @@
     <xacro:iris_inertial/>
   </link>
-  <joint name="${side}_camera_joint" type="fixed">
+  <!-- <joint name="${side}_camera_joint" type="fixed">
     <origin rpy="0 0 0" xyz="-0.001 0 0"/>
     <parent link="${side}_eyesupport_link"/>
     <child link="${side}_camera_link"/>
-  </joint>
+  </joint> -->
   <joint name="${side}_eye_joint" type="fixed">
     <origin rpy="0 0 0" xyz="0.003 0 0"/>

File: inmoov_description/urdf/asmFace.urdf.xacro (robot description, xacro)
@@ -13,7 +13,5 @@
     <xacro:face_inertial/>
   </link>
-  <joint name="eyes_tilt_joint" type="revolute">
-   <axis xyz="0 1 0"/>
-   <limit effort="1000.0" lower="${eyes_tilt_joint_lower}" upper="${eyes_tilt_joint_upper}" velocity="${eyes_tilt_joint_velocity}" />
+  <joint name="eyes_tilt_joint" type="fixed">
    <origin rpy="0 0 0" xyz="0 0 0"/>
    <parent link="face_link"/>
@@ -31,7 +29,5 @@
   </link>
 <xacro:asmEye side="r"/>
-  <joint name="eyes_pan_joint" type="revolute">
-   <axis xyz="0 0 1"/>
-    <limit effort="1000.0" lower="${eyes_pan_joint_lower}" upper="${eyes_pan_joint_upper}" velocity="${eyes_pan_joint_velocity}" />
+  <joint name="eyes_pan_joint" type="fixed">
    <origin rpy="0 0 0" xyz="0 0.033 -0.0036"/>
    <parent link="eyesupport_link"/>
@@ -39,8 +35,5 @@
   </joint>
 <xacro:asmEye side="l" />
-  <joint name="l_eye_pan_joint" type="revolute">
-   <axis xyz="0 0 1"/>
-   <limit effort="1000.0" lower="${eyes_pan_joint_lower}" upper="${eyes_pan_joint_upper}" velocity="${eyes_pan_joint_velocity}" />
-   <mimic joint="eyes_pan_joint" multiplier="1" offset="0"/>
+  <joint name="l_eye_pan_joint" type="fixed">
    <origin rpy="0 0 0" xyz="0 -0.033 -0.0036"/>
    <parent link="eyesupport_link"/>

File: inmoov_description/urdf/asmHead.urdf.xacro (robot description, xacro)
@@ -62,14 +62,10 @@
     <xacro:earrightv1_inertial/>
   </link>
-  <joint name="head_pan_joint" type="revolute">
-   <axis xyz="0 0 1"/>
-   <limit effort="1000.0" lower="${head_pan_joint_lower}" upper="${head_pan_joint_upper}" velocity="${head_pan_joint_velocity}" />
+  <joint name="head_pan_joint" type="fixed">
    <origin rpy="0 0 0" xyz="0 0 0.0245"/>
    <parent link="head_base_link"/>
    <child link="head_link"/>
   </joint>
-  <joint name="jaw_joint" type="revolute">
-   <axis xyz="0 1 0"/>
-   <limit effort="1000.0" lower="${jaw_joint_lower}" upper="${jaw_joint_upper}" velocity="${jaw_joint_velocity}" />
+  <joint name="jaw_joint" type="fixed">
    <origin rpy="0 0.09 0" xyz="0.0375 0.0005 0.0437"/>
    <parent link="head_link"/>

File: inmoov_description/urdf/asmTorso.urdf.xacro (robot description, xacro)
@@ -52,24 +52,4 @@
     <xacro:kinectone_inertial/>
   </link>
-  <link name="kinect2_ir_optical_frame">
-    <visual>
-      <geometry>
-        <mesh filename="package://inmoov_meshes/meshes/kinectone.stl" scale="0.001 0.001 0.001"/>
-      </geometry>
-      <origin rpy="1.57 0 0" xyz="0 0 0"/>
-      <xacro:kinect_color/>
-    </visual>
-    <xacro:kinectone_inertial/>
-  </link>
-  <link name="kinect2_rgb_optical_frame">
-    <visual>
-      <geometry>
-        <mesh filename="package://inmoov_meshes/meshes/kinectone.stl" scale="0.001 0.001 0.001"/>
-      </geometry>
-      <origin rpy="1.57 0 0" xyz="0 0 0"/>
-      <xacro:kinect_color/>
-    </visual>
-    <xacro:kinectone_inertial/>
-  </link>
   <link name="chestplate_link">
     <visual>
@@ -82,5 +62,5 @@
     <xacro:chest_inertial/>
   </link>
-  <joint name="waist_pan_joint" type="revolute">
+  <!-- <joint name="waist_pan_joint" type="revolute">
    <axis xyz="0 0 1"/>
    <limit effort="1000.0" lower="${waist_pan_joint_lower}" upper="${waist_pan_joint_upper}" velocity="${waist_pan_joint_velocity}" />
@@ -88,11 +68,16 @@
     <parent link="mid_stomach_link"/>
     <child link="top_stomach_link"/>
+  </joint> -->
+  <joint name="waist_pan_joint" type="fixed">
+    <origin rpy="0 0 0" xyz="0 0 1.152"/>
+    <parent link="mid_stomach_link"/>
+    <child link="top_stomach_link"/>
   </joint>
   <joint name="disk_joint" type="fixed">
-      <origin rpy="0 0 0" xyz="0.046 0 0.09"/>
+    <origin rpy="0 0 0" xyz="0.046 0 0.09"/>
     <parent link="top_stomach_link"/>
     <child link="disk_link"/>
   </joint>
-  <joint name="waist_roll_joint" type="revolute">
+  <!-- <joint name="waist_roll_joint" type="revolute">
    <axis xyz="1 0 0"/>
    <limit effort="1000.0" lower="${waist_roll_joint_lower}" upper="${waist_roll_joint_upper}" velocity="${waist_roll_joint_velocity}" />
@@ -100,25 +85,20 @@
     <parent link="top_stomach_link"/>
     <child link="torso_link"/>
+  </joint> -->
+  <joint name="waist_roll_joint" type="fixed">
+    <origin rpy="0 0 0" xyz="0 0 0.11"/>
+    <parent link="top_stomach_link"/>
+    <child link="torso_link"/>
   </joint>
   <joint name="chestplate_joint" type="fixed">
-<origin rpy="0 0 0" xyz="0.042 0 0.025"/>
+    <origin rpy="0 0 0" xyz="0.042 0 0.025"/>
     <parent link="torso_link"/>
     <child link="chestplate_link"/>
   </joint>
   <joint name="kinect2_joint" type="fixed">
-<origin rpy="-1.57 0 -1.57" xyz="0 0 0.066"/>
+    <origin rpy="-1.57 0 -1.57" xyz="0 0 0.066"/>
     <parent link="torso_link"/>
     <child link="kinect2_link"/>
   </joint>
-  <joint name="kinect2_ir_optical_frame_joint" type="fixed">
-<origin rpy="-1.57 0 -1.57" xyz="0 0 0.066"/>
-    <parent link="torso_link"/>
-    <child link="kinect2_ir_optical_frame"/>
-  </joint>
-  <joint name="kinect2_rgb_optical_joint" type="fixed">
-<origin rpy="-1.57 0 -1.57" xyz="0 0 0.066"/>
-    <parent link="torso_link"/>
-    <child link="kinect2_rgb_optical_frame"/>
-  </joint>
 </xacro:macro>
 </robot>
