Commit message: fix wrist in hand skeleton

File: inmoov_description/robots/inmoov_right_hand.urdf (robot description, URDF)
Before this commit: robot inmoov_hand, 27 links, 26 joints
Joints:
- joint base_to_hand_joint: axis 0 0 1 -> (none); limit lower=-3.14 upper=0 effort=1000.0 velocity=0.5 -> (none); type revolute -> fixed

File: inmoov_description/robots/inmoov_right_hand.urdf.xacro (robot description, xacro)
@@ -17,8 +17,6 @@
   </link>
   <xacro:hand side="r" flip="1" covers="yes" />
-  <joint name="base_to_hand_joint" type="revolute">
-   <axis xyz="0 0 1"/>
-<limit effort="1000.0" lower="-3.14" upper="0" velocity="0.5"/>
-<origin rpy="0 0 0" xyz="0 0 0"/>
+  <joint name="base_to_hand_joint" type="fixed">
+    <origin rpy="0 0 0" xyz="0 0 0"/>
     <parent link="base_link"/>
     <child link="r_hand_link"/>
