Commit message: mods ikfast why

File: inmoov_description/robots/inmoov_shadow_hand.urdf (robot description, URDF)
Before this commit: robot inmoov, 70 links, 69 joints
Links:
- added link l_forearm_link_aux
- added link r_forearm_link_aux
Joints:
- added joint l_elbow_roll_joint: type revolute, parent l_forearm_link_aux, child l_forearm_link, origin xyz=0.0 0 0.0 rpy=0 0 0, axis 0 0 1, limit lower=-3.14159265359 upper=3.14159265359 effort=1000.0 velocity=1745.32925199
- added joint r_elbow_roll_joint: type revolute, parent r_forearm_link_aux, child r_forearm_link, origin xyz=0.0 0 0.0 rpy=0 0 0, axis 0 0 1, limit lower=-1.57079632679 upper=1.57079632679 effort=1000.0 velocity=1745.32925199
- joint l_elbow_flex_joint: child l_forearm_link -> l_forearm_link_aux; origin xyz=-0.0278 0 -0.2235 rpy=0 0 0 -> xyz=-0.03 0 -0.225 rpy=0 0 0
- joint l_shoulder_out_joint: origin xyz=0 0.143 0.298 rpy=0 0 0 -> xyz=0 0.14 0.3 rpy=0 0 0
- joint l_upper_arm_roll_joint: origin xyz=0 0.066 -0.060 rpy=0 0 0 -> xyz=0 0.066 -0.06 rpy=0 0 0
- joint r_elbow_flex_joint: child r_forearm_link -> r_forearm_link_aux; limit lower=-3.14159265359 upper=3.14159265359 effort=1000.0 velocity=1745.32925199 -> lower=-1.57079632679 upper=1.57079632679 effort=1000.0 velocity=1745.32925199; origin xyz=-0.0278 0 -0.2235 rpy=0 0 0 -> xyz=-0.03 0 -0.225 rpy=0 0 0
- joint r_shoulder_lift_joint: limit lower=-3.14159265359 upper=3.14159265359 effort=1000.0 velocity=1745.32925199 -> lower=-1.57079632679 upper=1.57079632679 effort=1000.0 velocity=1745.32925199
- joint r_shoulder_out_joint: limit lower=-3.14159265359 upper=3.14159265359 effort=1000.0 velocity=1745.32925199 -> lower=-3.14159265359 upper=0 effort=1000.0 velocity=1745.32925199; origin xyz=0 -0.143 0.298 rpy=0 0 0 -> xyz=0 -0.14 0.3 rpy=0 0 0
- joint r_upper_arm_roll_joint: limit lower=-3.14159265359 upper=3.14159265359 effort=1000.0 velocity=1745.32925199 -> lower=-1.57079632679 upper=1.57079632679 effort=1000.0 velocity=1745.32925199; origin xyz=0 -0.066 -0.060 rpy=0 0 0 -> xyz=0 -0.066 -0.06 rpy=0 0 0
- joint r_wrist_roll_joint: axis 0 0 1 -> (none); limit lower=-3.14159265359 upper=3.14159265359 effort=1000.0 velocity=1745.32925199 -> (none); origin xyz=-0.0144 0.01  -0.2885 rpy=3.14 0 0 -> xyz=-0.015 0.01  -0.3 rpy=3.14159265359 0 0; type revolute -> fixed
- joint rh_WRJ1: limit lower=-0.698131700798 upper=0.488692190558 effort=30 velocity=2.0 -> lower=-1.57079632679 upper=1.57079632679 effort=30 velocity=2.0; origin xyz=0 0 0.034 rpy=0 0 0 -> xyz=0 0 0.03 rpy=0 0 0
- joint rh_WRJ2: limit lower=-0.523598775598 upper=0.174532925199 effort=10 velocity=2.0 -> lower=-1.57079632679 upper=1.57079632679 effort=10 velocity=2.0; origin xyz=0 -0.010 0.0 rpy=0 0 0 -> xyz=0 0.0 0.0 rpy=0 0 0

File: inmoov_description/robots/inmoov_shadow_hand.urdf.xacro (robot description, xacro)
@@ -84,5 +84,5 @@
    <axis xyz="1 0 0"/>
    <limit effort="1000.0" lower="${r_shoulder_out_joint_lower}" upper="${r_shoulder_out_joint_upper}" velocity="${r_shoulder_out_joint_velocity}" />
-   <origin rpy="0 0 0" xyz="0 -0.143 0.298"/>
+   <origin rpy="0 0 0" xyz="0 -0.14 0.3"/>
    <parent link="torso_link"/>
    <child link="r_shoulder_base_link"/>
@@ -100,5 +100,5 @@
     <!-- hand with cylindrical base drifts in gazebo, attach it to the world -->
     <link name="r_hand_link" />
-    <joint name="r_wrist_roll_joint" type="revolute">
+    <!-- <joint name="r_wrist_roll_joint" type="revolute">
         <axis xyz="0 0 1"/>
         <limit effort="1000.0" lower="${r_wrist_roll_joint_lower}" upper="${r_wrist_roll_joint_upper}" velocity="${r_wrist_roll_joint_velocity}" />
@@ -106,4 +106,10 @@
         <child link="r_hand_link" />
         <origin rpy="3.14 0 0" xyz="-0.0144 0.01  -0.2885"/>
+    </joint> -->
+    <!-- move wrist roll to elbow roll for now -->
+    <joint name="r_wrist_roll_joint" type="fixed">
+        <parent link="r_forearm_link" />
+        <child link="r_hand_link" />
+        <origin rpy="3.14159265359 0 0" xyz="-0.015 0.01  -0.3"/>
     </joint>
     <xacro:shadowhand muscletrans="false" muscle="false" hand_type="hand_e" bio="false" bt_sp="false"
@@ -113,5 +119,5 @@
    <axis xyz="1 0 0"/>
    <limit effort="1000.0" lower="${l_shoulder_out_joint_lower}" upper="${l_shoulder_out_joint_upper}" velocity="${l_shoulder_out_joint_velocity}" />
-   <origin rpy="0 0 0" xyz="0 0.143 0.298"/>
+   <origin rpy="0 0 0" xyz="0 0.14 0.3"/>
    <parent link="torso_link"/>
    <child link="l_shoulder_base_link"/>

File: inmoov_description/urdf/asmArm.urdf.xacro (robot description, xacro)
@@ -52,4 +52,5 @@
     <xacro:bicepcover_inertial/>
   </link>
+  <link name="${side}_forearm_link_aux"/>
   <link name="${side}_forearm_link">
     <visual>
@@ -87,5 +88,5 @@
       <limit effort="1000.0" lower="${r_upper_arm_roll_joint_lower}" upper="${r_upper_arm_roll_joint_upper}" velocity="${r_upper_arm_roll_joint_velocity}" />
     </xacro:if>
-    <origin rpy="0 0 0" xyz="0 ${flip * -0.066} -0.060"/>
+    <origin rpy="0 0 0" xyz="0 ${flip * -0.066} -0.06"/>
     <parent link="${side}_shoulder_link"/>
     <child link="${side}_bicep_link"/>
@@ -99,6 +100,18 @@
       <limit effort="1000.0" lower="${r_elbow_flex_joint_lower}" upper="${r_elbow_flex_joint_upper}" velocity="${r_elbow_flex_joint_velocity}" />
     </xacro:if>
-    <origin rpy="0 0 0" xyz="-0.0278 0 -0.2235"/>
+    <origin rpy="0 0 0" xyz="-0.03 0 -0.225"/>
     <parent link="${side}_bicep_link"/>
+    <child link="${side}_forearm_link_aux"/>
+  </joint>
+  <joint name="${side}_elbow_roll_joint" type="revolute">
+    <axis xyz="0 0 1"/>
+    <xacro:if value="${side == 'l'}">
+      <limit effort="1000.0" lower="${l_wrist_roll_joint_lower}" upper="${l_wrist_roll_joint_upper}" velocity="${l_wrist_roll_joint_velocity}" />
+    </xacro:if>
+    <xacro:if value="${side == 'r'}">
+      <limit effort="1000.0" lower="${r_wrist_roll_joint_lower}" upper="${r_wrist_roll_joint_upper}" velocity="${r_wrist_roll_joint_velocity}" />
+    </xacro:if>
+    <origin rpy="0 0 0" xyz="0.0 0 0.0"/>
+    <parent link="${side}_forearm_link_aux"/>
     <child link="${side}_forearm_link"/>
   </joint>

Commit message: realitic mods RoM and forarm collision

File: inmoov_description/robots/inmoov_shadow_hand.urdf (robot description, URDF)
Before this commit: robot inmoov, 72 links, 71 joints
Links:
- link l_forearm_link: geometry collision cylinder length=0.28 radius=0.045; visual mesh filename=package://inmoov_meshes/meshes/l_forearm.stl scale=0.001 0.001 0.001
- link l_hand_link: geometry 
- link r_forearm_link: geometry collision cylinder length=0.28 radius=0.045; visual mesh filename=package://inmoov_meshes/meshes/r_forearm.stl scale=0.001 0.001 0.001
Joints:
- joint l_elbow_flex_joint: limit lower=-3.14159265359 upper=3.14159265359 effort=1000.0 velocity=1745.32925199 -> lower=-3.14159265359 upper=0.0 effort=1000.0 velocity=1745.32925199
- joint l_elbow_roll_joint: limit lower=-3.14159265359 upper=3.14159265359 effort=1000.0 velocity=1745.32925199 -> lower=-1.57079632679 upper=1.57079632679 effort=1000.0 velocity=1745.32925199
- joint l_shoulder_lift_joint: limit lower=-3.14159265359 upper=3.14159265359 effort=1000.0 velocity=1745.32925199 -> lower=-1.57079632679 upper=1.57079632679 effort=1000.0 velocity=1745.32925199
- joint l_shoulder_out_joint: limit lower=-3.14159265359 upper=3.14159265359 effort=1000.0 velocity=1745.32925199 -> lower=-1.57079632679 upper=1.57079632679 effort=1000.0 velocity=1745.32925199
- joint l_upper_arm_roll_joint: limit lower=-3.14159265359 upper=3.14159265359 effort=1000.0 velocity=1745.32925199 -> lower=-1.57079632679 upper=1.57079632679 effort=1000.0 velocity=1745.32925199
- joint l_wrist_roll_joint: axis 0 0 1 -> (none); limit lower=-3.14159265359 upper=3.14159265359 effort=1000.0 velocity=1745.32925199 -> (none); origin xyz=-0.0144 -0.01  -0.2885 rpy=0 0 0 -> xyz=-0.015 0.01  -0.3 rpy=3.14159265359 0 0; type revolute -> fixed
- joint r_elbow_flex_joint: limit lower=-1.57079632679 upper=1.57079632679 effort=1000.0 velocity=1745.32925199 -> lower=-3.14159265359 upper=0.0 effort=1000.0 velocity=1745.32925199
- joint r_shoulder_out_joint: limit lower=-3.14159265359 upper=0 effort=1000.0 velocity=1745.32925199 -> lower=-1.57079632679 upper=1.57079632679 effort=1000.0 velocity=1745.32925199
- joint rh_WRJ1: limit lower=-1.57079632679 upper=1.57079632679 effort=30 velocity=2.0 -> lower=-1.57079632679 upper=1.57079632679 effort=30 velocity=20.0
- joint rh_WRJ2: limit lower=-1.57079632679 upper=1.57079632679 effort=10 velocity=2.0 -> lower=-1.0471975512 upper=1.0471975512 effort=10 velocity=20.0

File: inmoov_description/robots/inmoov_shadow_hand.urdf.xacro (robot description, xacro)
@@ -12,7 +12,9 @@
   <xacro:include filename="$(find inmoov_description)/urdf/asmFace.urdf.xacro" />
   <xacro:include filename="$(find inmoov_description)/urdf/asmArm.urdf.xacro" />
-    <xacro:include filename="$(find sr_description)/materials.urdf.xacro"/>
-    <xacro:include filename="$(find sr_description)/hand/xacro/full_hand.urdf.xacro"/>
-    <xacro:include filename="$(find sr_description)/other/xacro/gazebo/gazebo.urdf.xacro"/>
+  <xacro:include filename="$(find sr_description)/materials.urdf.xacro"/>
+  <xacro:include filename="$(find sr_description)/hand/xacro/full_hand.urdf.xacro"/>
+  <xacro:include filename="$(find sr_description)/other/xacro/gazebo/gazebo.urdf.xacro"/>
+  <xacro:property name="M_PI" value="3.1415926535897931" />
+  <!-- usage: e.g. ${M_PI/4} -->
   <link name="world"/>
   <joint name="fixed" type="fixed">
@@ -88,31 +90,22 @@
    <child link="r_shoulder_base_link"/>
   </joint>
-  <!-- <link name="r_hand_link">
-    <visual>
-      <geometry>
-        <cylinder length="0.11" radius="0.06"/>
-      </geometry>
-      <origin rpy="0 0 0" xyz="0 0 0.055"/>
-      <xacro:base_color/>
-    </visual>
-  </link> -->
   <!-- shadow hand -->
-    <!-- hand with cylindrical base drifts in gazebo, attach it to the world -->
-    <link name="r_hand_link" />
-    <!-- <joint name="r_wrist_roll_joint" type="revolute">
-        <axis xyz="0 0 1"/>
-        <limit effort="1000.0" lower="${r_wrist_roll_joint_lower}" upper="${r_wrist_roll_joint_upper}" velocity="${r_wrist_roll_joint_velocity}" />
-        <parent link="r_forearm_link" />
-        <child link="r_hand_link" />
-        <origin rpy="3.14 0 0" xyz="-0.0144 0.01  -0.2885"/>
-    </joint> -->
-    <!-- move wrist roll to elbow roll for now -->
-    <joint name="r_wrist_roll_joint" type="fixed">
-        <parent link="r_forearm_link" />
-        <child link="r_hand_link" />
-        <origin rpy="3.14159265359 0 0" xyz="-0.015 0.01  -0.3"/>
-    </joint>
-    <xacro:shadowhand muscletrans="false" muscle="false" hand_type="hand_e" bio="false" bt_sp="false"
-                      ubi="false" eli="false" reflect="1.0" prefix="rh_" lf="true" parent="r_hand_link"/>
+  <!-- hand with cylindrical base drifts in gazebo, attach it to the world -->
+  <link name="r_hand_link" />
+  <!-- <joint name="r_wrist_roll_joint" type="revolute">
+      <axis xyz="0 0 1"/>
+      <limit effort="1000.0" lower="${r_wrist_roll_joint_lower}" upper="${r_wrist_roll_joint_upper}" velocity="${r_wrist_roll_joint_velocity}" />
+      <parent link="r_forearm_link" />
+      <child link="r_hand_link" />
+      <origin rpy="3.14 0 0" xyz="-0.0144 0.01  -0.2885"/>
+  </joint> -->
+  <!-- move wrist roll to elbow roll for now -->
+  <joint name="r_wrist_roll_joint" type="fixed">
+      <parent link="r_forearm_link" />
+      <child link="r_hand_link" />
+      <origin rpy="${M_PI} 0 0" xyz="-0.015 0.01  -0.3"/>
+  </joint>
+  <xacro:shadowhand muscletrans="false" muscle="false" hand_type="hand_e" bio="false" bt_sp="false"
+                    ubi="false" eli="false" reflect="1.0" prefix="rh_" lf="true" parent="r_hand_link"/>
   <xacro:arm side="l" flip="-1" covers="yes" />
   <joint name="l_shoulder_out_joint" type="revolute">
@@ -123,17 +116,7 @@
    <child link="l_shoulder_base_link"/>
   </joint>
-  <link name="l_hand_link">
-    <visual>
-      <geometry>
-        <cylinder length="0.11" radius="0.06"/>
-      </geometry>
-      <origin rpy="0 0 0" xyz="0 0 0.055"/>
-      <xacro:base_color/>
-    </visual>
-  </link>
-  <joint name="l_wrist_roll_joint" type="revolute">
-   <axis xyz="0 0 1"/>
-   <limit effort="1000.0" lower="${l_wrist_roll_joint_lower}" upper="${l_wrist_roll_joint_upper}" velocity="${l_wrist_roll_joint_velocity}" />
-   <origin rpy="0 0 0" xyz="-0.0144 -0.01  -0.2885"/>
+  <link name="l_hand_link" />
+  <joint name="l_wrist_roll_joint" type="fixed">
+   <origin rpy="${M_PI} 0 0" xyz="-0.015 0.01  -0.3"/>
    <parent link="l_forearm_link"/>
    <child link="l_hand_link"/>

File: inmoov_description/urdf/asmArm.urdf.xacro (robot description, xacro)
@@ -1,4 +1,6 @@
 <?xml version="1.0"?>
 <robot name="inmoov" xmlns:xacro="http://ros.org/wiki/xacro">
+ <xacro:property name="M_PI" value="3.1415926535897931" />
+ <!-- usage: e.g. ${M_PI/4} -->
 <xacro:macro name="arm" params="side flip covers">
   <link name="${side}_shoulder_base_link">
@@ -61,4 +63,10 @@
       <xacro:cover_color/>
     </visual>
+    <collision>
+      <geometry>
+        <cylinder length="0.28" radius="0.045"/>
+      </geometry>
+      <origin rpy="0 0 0" xyz="-0.00 0 -0.14"/>
+    </collision>
     <xacro:if value="${side == 'l'}">
       <xacro:l_forearm_inertial/>

Commit message: add inmoov shadow hand env

File: inmoov_description/robots/inmoov_shadow_hand.urdf (robot description, URDF)
Before this commit: robot inmoov, 72 links, 71 joints
Joints:
- joint waist_pan_joint: type revolute -> fixed
- joint waist_roll_joint: type revolute -> fixed

Commit message: disable forearm collision

File: inmoov_description/robots/inmoov_shadow_hand.urdf (robot description, URDF)
Before this commit: robot inmoov, 72 links, 71 joints
Links:
- link l_forearm_link: geometry visual mesh filename=package://inmoov_meshes/meshes/l_forearm.stl scale=0.001 0.001 0.001
- link r_forearm_link: geometry visual mesh filename=package://inmoov_meshes/meshes/r_forearm.stl scale=0.001 0.001 0.001
