Commit message: remove unused link manipulator

File: inmoov_description/robots/inmoov_shadow_hand_v2.urdf (robot description, URDF)
Before this commit: robot inmoov, 72 links, 71 joints
Links:
- removed link rh_manipulator
Joints:
- removed joint rh_ee_fixed_joint

Commit message: collada fix

File: inmoov_description/robots/inmoov_shadow_hand_v2.urdf (robot description, URDF)
Before this commit: robot inmoov, 72 links, 71 joints
Links:
- removed link world
Joints:
- removed joint fixed
- joint base_to_pedestal_link: origin xyz=0 0 0 rpy=0 0 0 -> xyz=0 0 0.58 rpy=0 0 0
- joint pedestal_to_mid_stomach_joint: origin xyz=0 0 0 rpy=0 0 0 -> xyz=0 0 0.572 rpy=0 0 0
- joint waist_pan_joint: origin xyz=0 0 1.152 rpy=0 0 0 -> xyz=0 0 0 rpy=0 0 0
