Commit message: mods according to artist

File: inmoov_description/robots/inmoov_shadow_hand_v2_1.urdf (robot description, URDF)
Before this commit: robot inmoov, 72 links, 71 joints
Joints:
- joint r_elbow_flex_joint: origin xyz=-0.03 0 -0.225 rpy=0 0 0 -> xyz=-0.054 -0.009 -0.2621 rpy=0 0 0
- joint r_wrist_roll_joint: origin xyz=-0.015 0.01 -0.3 rpy=3.14159265359 0 0 -> xyz=0.0303 -0.00729 -0.302 rpy=3.14159265359 0 0
