Commit message: init using comfotrable pose, place with cyl & with hand collision on

File: inmoov_description/robots/inmoov_arm_v2_2_obj.urdf (robot description, URDF)
Before this commit: robot inmoov, 11 links, 10 joints
Links:
- link obj: geometry collision box size=0.08 0.08 0.20; visual box size=0.08 0.08 0.20
- link obj_z: mass None -> 1
Joints:
- joint rh_obj_j: origin xyz=-0.11985664814710617, -0.15380138158798218, 0.13343362510204315 rpy=-1.5708 0.2292 -1.5708 -> xyz=-0.10985665023326874, -0.15379363298416138, 0.1334318220615387 rpy=-1.570982165314285 -0.22920366351116048 -1.5699785493771878
