Commit message: enlarge shoulder jl a bit

File: inmoov_description/robots/inmoov_arm_v2_2_reaching_BB.urdf (robot description, URDF)
Before this commit: robot inmoov, 9 links, 8 joints
Joints:
- joint r_shoulder_lift_joint: limit lower=-1.57079632679 upper=1.57079632679 effort=1000.0 velocity=1745.32925199 -> lower=-2.07079632679 upper=1.57079632679 effort=1000.0 velocity=1745.32925199
- joint r_shoulder_out_joint: limit lower=-1.57079632679 upper=1.57079632679 effort=1000.0 velocity=1745.32925199 -> lower=-2.07079632679 upper=1.57079632679 effort=1000.0 velocity=1745.32925199

File: inmoov_description/robots/inmoov_shadow_hand_v2_2.urdf (robot description, URDF)
Before this commit: robot inmoov, 36 links, 35 joints
Joints:
- joint r_shoulder_lift_joint: limit lower=-1.57079632679 upper=1.57079632679 effort=1000.0 velocity=1745.32925199 -> lower=-2.07079632679 upper=1.57079632679 effort=1000.0 velocity=1745.32925199
- joint r_shoulder_out_joint: limit lower=-1.57079632679 upper=1.57079632679 effort=1000.0 velocity=1745.32925199 -> lower=-2.07079632679 upper=1.57079632679 effort=1000.0 velocity=1745.32925199
