Commit message: enlarge finger range and use ellipsoid collision shape

File: inmoov_description/robots/inmoov_shadow_hand_v2_2.urdf (robot description, URDF)
Before this commit: robot inmoov, 36 links, 35 joints
Links:
- link rh_ffdistal: geometry collision mesh filename=package://sr_description/hand/model/ellipsoids/distal_ellip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 scale=0.001 0.001 0.001; visual mesh filename=package://sr_description/hand/model/F1.dae scale=0.001 0.001 0.001
- link rh_lfdistal: geometry collision mesh filename=package://sr_description/hand/model/ellipsoids/distal_ellip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 scale=0.001 0.001 0.001; visual mesh filename=package://sr_description/hand/model/F1.dae scale=0.001 0.001 0.001
- link rh_mfdistal: geometry collision mesh filename=package://sr_description/hand/model/ellipsoids/distal_ellip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 scale=0.001 0.001 0.001; visual mesh filename=package://sr_description/hand/model/F1.dae scale=0.001 0.001 0.001
- link rh_rfdistal: geometry collision mesh filename=package://sr_description/hand/model/ellipsoids/distal_ellip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 scale=0.001 0.001 0.001; visual mesh filename=package://sr_description/hand/model/F1.dae scale=0.001 0.001 0.001
- link rh_thdistal: geometry collision mesh filename=package://sr_description/hand/model/ellipsoids/thdistal_ell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 scale=0.001 0.001 0.001; visual mesh filename=package://sr_description/hand/model/TH1_z.dae scale=0.001 0.001 0.001
Joints:
- joint rh_THJ2: limit lower=-0.698131700798 upper=0.698131700798 effort=2.0 velocity=2.0 -> lower=-0.698131700798 upper=1.2217304764 effort=2.0 velocity=2.0
- joint rh_THJ4: limit lower=0.0 upper=1.2217304764 effort=3 velocity=4.0 -> lower=0.0 upper=2.01 effort=3 velocity=4.0

Commit message: add collision to lower arm

File: inmoov_description/robots/inmoov_shadow_hand_v2_2.urdf (robot description, URDF)
Before this commit: robot inmoov, 36 links, 35 joints
Links:
- link r_forearm_link: geometry collision box size=0.06 0.06 0.2; visual box size=0.06 0.06 0.2

Commit message: mods placing open up

File: inmoov_description/robots/inmoov_shadow_hand_v2_2.urdf (robot description, URDF)
Before this commit: robot inmoov, 36 links, 35 joints
Links:
- link rh_wrist: geometry visual mesh filename=package://sr_description/hand/model/wrist.dae scale=0.001 0.001 0.001

Commit message: revert jl

File: inmoov_description/robots/inmoov_shadow_hand_v2_2.urdf (robot description, URDF)
Before this commit: robot inmoov, 36 links, 35 joints
Joints:
- joint rh_THJ2: limit lower=-0.698131700798 upper=1.2217304764 effort=2.0 velocity=2.0 -> lower=-0.698131700798 upper=0.6917304764 effort=2.0 velocity=2.0
- joint rh_THJ4: limit lower=0.0 upper=2.01 effort=3 velocity=4.0 -> lower=0.0 upper=1.2217304764 effort=3 velocity=4.0
