Commit message: planning BB urdfs with hacks

File: inmoov_description/robots/inmoov_arm_v2_2_moving_BB.urdf (robot description, URDF)
Before this commit: robot inmoov, 9 links, 8 joints
Links:
- link r_forearm_link: geometry collision box size=0.08 0.08 0.22; visual mesh filename=package://inmoov_meshes/meshes/r_forearm.stl scale=0.001 0.001 0.001
- link rh_palm: geometry collision box size=0.18 0.15 0.18; visual box size=0.18 0.15 0.18

Commit message: mod arms for openrave viz

File: inmoov_description/robots/inmoov_arm_v2_2_moving_BB.urdf (robot description, URDF)
Before this commit: robot inmoov, 9 links, 8 joints
Links:
- link r_forearm_link: geometry collision box size=0.07 0.07 0.2; visual mesh filename=package://inmoov_meshes/meshes/box-binary.stl scale=0.07 0.07 0.2
- link rh_palm: geometry collision box size=0.18 0.15 0.18; visual mesh filename=package://inmoov_meshes/meshes/box-binary.stl scale=0.18 0.15 0.18
- link rh_wrist: geometry visual mesh filename=package://sr_description/hand/model/wrist.dae scale=0.001 0.001 0.001

File: inmoov_description/robots/inmoov_arm_v2_2_reaching_BB.urdf (robot description, URDF)
Before this commit: robot inmoov, 9 links, 8 joints
Links:
- link r_forearm_link: geometry collision box size=0.07 0.07 0.2; visual mesh filename=package://inmoov_meshes/meshes/box-binary.stl scale=0.07 0.07 0.2
- link rh_palm: geometry collision box size=0.10 0.10 0.18; visual mesh filename=package://inmoov_meshes/meshes/box-binary.stl scale=0.10 0.10 0.18
- link rh_wrist: geometry visual mesh filename=package://sr_description/hand/model/wrist.dae scale=0.001 0.001 0.001

File: inmoov_description/robots/inmoov_shadow_hand_v2_2.urdf (robot description, URDF)
Before this commit: robot inmoov, 36 links, 35 joints
Links:
- link r_forearm_link: geometry collision box size=0.06 0.06 0.2; visual mesh filename=package://inmoov_meshes/meshes/box-binary.stl scale=0.06 0.06 0.2
